File: SG4000_SendRtrn_Balun.kicad_pcb (KiCad board)
At the start: 2 copper layers, 40 parts, among them J1001 Power Entry, J1002 Audio to MB, J1003 Audio To XLR, U1001 NE5532AP, U1002 NE5534AP

Commit message: Add files via upload
Parts:
- moved U1001 101.8 mm to (225.4, 52.7), turned to 270 degrees
- moved R1011 31.0 mm to (262.3, 52.1)
- moved J1003 27.8 mm to (276.9, 80.6)
- moved C1019 21.1 mm to (249.6, 76.8), turned to 90 degrees
- moved C1022 20.7 mm to (261.0, 57.1), turned to 270 degrees
- moved C1020 20.4 mm to (261.0, 72.4), turned to 270 degrees
- moved C1021 19.8 mm to (249.6, 61.6), turned to 90 degrees
- moved R1012 17.1 mm to (272.4, 82.5)
- moved R1013 16.8 mm to (271.1, 78.1), turned to 90 degrees
- moved R1010 10.6 mm to (262.3, 67.3)

Commit message: Add files via upload
Parts:
- moved J1001 183.1 mm to (223.5, 134.6), turned to 90 degrees
- moved C1004 166.6 mm to (229.9, 114.3), turned to 0 degrees
- moved C1003 159.9 mm to (221.0, 114.3), turned to 0 degrees
- moved C1002 156.8 mm to (229.9, 125.7), turned to 0 degrees
- moved C1001 151.0 mm to (221.0, 125.7), turned to 0 degrees
- moved J1002 137.8 mm to (174.0, 69.2)
- moved C1005 72.6 mm to (130.4, 137.7)
- moved C1016 72.6 mm to (112.6, 158.9)
- moved C1009 72.6 mm to (122.0, 141.6)
- moved C1010 72.6 mm to (113.0, 150.8)
- moved C1011 72.6 mm to (72.0, 159.0)
- moved C1013 72.6 mm to (104.6, 152.8)
- moved C1015 72.6 mm to (113.3, 131.2)
- moved C1017 72.6 mm to (121.0, 149.8)
- moved R1003 72.6 mm to (66.7, 152.0)
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
Commit message: Add files via upload
Parts:
- moved J1003 124.9 mm to (155.6, 90.8)
- moved R1013 123.2 mm to (155.6, 120.7)
- moved C1022 120.1 mm to (148.0, 97.8)
- moved C1019 120.1 mm to (136.5, 117.5)
- moved C1020 120.1 mm to (148.0, 113.0)
- moved C1021 120.1 mm to (136.5, 102.2)
- moved R1011 120.1 mm to (149.2, 92.7)
- moved R1010 118.3 mm to (151.1, 108.0)
- moved R1012 117.7 mm to (155.6, 96.5), turned to 270 degrees
- moved U1001 116.7 mm to (120.7, 104.1)
- moved R1003 112.6 mm to (141.0, 67.3), turned to 270 degrees
- moved C1003 110.1 mm to (111.8, 128.3), turned to 90 degrees
- moved R1004 101.4 mm to (132.1, 67.3), turned to 270 degrees
- moved C1001 100.4 mm to (120.7, 128.3), turned to 90 degrees
- moved C1012 99.1 mm to (123.2, 77.5), turned to 90 degrees
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Other:
- board outline added: 58.4 x 76.2 mm
- net class Audio added: clearance 0.508, trace_width 0.508, via_dia 685.8, via_drill 0.3302
- net class Default: clearance 0.2 -> 0.508; trace_width 0.25 -> 0.508; via_dia 0.6 -> 0.6858; via_drill 0.4 -> 0.3302
- net class GND added: clearance 0.762, trace_width 0.762, via_dia 0.6858, via_drill 0.3302
- net class Power Rail added: clearance 0.762, trace_width 0.762, via_dia 0.6858, via_drill 0.3302
- net class Signal added: clearance 0.508, trace_width 0.508, via_dia 0.6858, via_drill 0.4
- rule trace_clearance: 0.2 -> 0.508
- rule via_min_drill: 0.3 -> 0.3302
- rule via_min_size: 0.4 -> 0.6858

Commit message: Add files via upload
Parts:
- moved C1017 160.6 mm to (266.9, 102.2)
- moved C1011 149.3 mm to (253.6, 130.8)
- moved C1020 118.4 mm to (266.2, 107.8)
- moved R1011 112.1 mm to (261.0, 101.6)
- moved R1007 108.0 mm to (212.8, 129.4)
- moved R1009 107.1 mm to (229.4, 121.3)
- moved C1022 101.8 mm to (241.3, 138.4)
- moved R1013 101.6 mm to (257.2, 117.6)
- moved R1006 100.7 mm to (227.4, 115.5)
- moved R1010 100.7 mm to (251.5, 115.5)
- moved R1001 100.2 mm to (221.6, 109.8)
- moved R1002 95.1 mm to (207.0, 130.4)
- moved R1012 85.3 mm to (237.2, 121.3)
- moved C1019 75.0 mm to (210.5, 104.7)
- moved C1021 75.0 mm to (210.5, 114.9)
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Other:
- board size 58.4 x 76.2 mm -> 88.9 x 63.5 mm

Commit message: Add files via upload
Parts:
- moved C1005 181.3 mm to (286.1, 62.5)
- moved C1015 176.8 mm to (278.7, 71.0)
- moved C1007 170.5 mm to (284.4, 42.1)
- moved C1018 160.9 mm to (266.2, 59.5), turned to 270 degrees
- moved C1014 160.2 mm to (260.2, 70.3)
- moved C1008 159.4 mm to (269.9, 76.3)
- moved C1013 156.3 mm to (273.4, 64.4), turned to 0 degrees
- moved C1016 149.1 mm to (270.7, 82.5)
- moved R1005 149.1 mm to (246.9, 43.0)
- moved R1008 149.0 mm to (257.1, 47.2)
- moved R1004 133.8 mm to (235.8, 56.3)
- moved C1006 126.9 mm to (250.1, 72.8)
- moved R1003 117.2 mm to (221.7, 67.8)
- moved C1002 109.8 mm to (266.2, 50.9)
- moved C1012 101.1 mm to (222.9, 87.4)
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Other:
- net class Audio: via_dia 685.8 -> 0.6858
- net class GND: clearance 0.762 -> 0.508; trace_width 0.762 -> 0.508
- net class Power Rail: clearance 0.762 -> 0.508; trace_width 0.762 -> 0.508
- board text added: "+15V"
- board text added: "+R"
- board text added: "+S"
- board text added: "-15V"
- board text added: "-R"
- board text added: "-S"
- board text added: "0V"
- board text added: "AUDIO TO MB"
- board text added: "AUDIO TO XLR"
- board text added: "RTN"
- board text added: "S"
